Commit message: Fixed tf issues

File: urdf/ur5e_robot.urdf.xacro (robot description, xacro)
@@ -12,4 +12,5 @@
     <!-- Here is where you define the scene and how the cframes are related -->
     <link name="world" />
+    <link name="palm" />
     <!-- Describe the interface between the robot and the gripper -->
     <joint name="robotiq_coupler_joint" type="fixed">
@@ -41,3 +42,10 @@
     <origin xyz="0.355 0.357 0.86" rpy="0.0 0.0 3.1416" />
     </joint>
+    <!-- Describe the location of the palm -->
+    <joint name="hand_palm" type="fixed">
+    <parent link="tool0" />
+    <child link="palm" />
+<!--        <origin xyz="0 0 0.13" rpy="0 0 0.2618 " />      &lt;!&ndash; Add in Z the hand's thickness (approx 13cm) &ndash;&gt;-->
+    <origin xyz="0 0 0.165" rpy="0 0 0.2618 " />      <!-- Add in Z the hand's thickness (approx 13cm) -->
+    </joint>
 </robot>

Commit message: Updated distances between cframes in the lab

File: urdf/ur5e_robot.urdf.xacro (robot description, xacro)
@@ -18,4 +18,5 @@
     <child link="lisas_hand" />
     <origin xyz="-0.0675 0.0675 0.004" rpy="0 0 ${-pi/2.0}" />
+        <!-- Note: x and y offset is because the cframe of the 3d model is not located in the center -->
     </joint>
     <!-- Describe the interface between the world and the tables -->
@@ -28,5 +29,7 @@
     <parent link="world" />
     <child link="small_table" />
-    <origin xyz="-0.21 -1.32 0" rpy="0 0 1.5708" />
+    <origin xyz="-0.23 -1.335 0" rpy="0 0 1.5708" />
+        <!-- x_offset = 1.715 - 1.845 = -.23  distances from next wall -->
+        <!-- y_offset = -1.335 -->
     </joint>
     <!-- Describe the interface between the world and the Apple Proxy -->
@@ -40,5 +43,5 @@
     <parent link="small_table" />
     <child link = "base_link" />
-    <origin xyz="0.355 0.357 0.86" rpy="0.0 0.0 3.1416" />
+    <origin xyz="0.358 0.357 0.858" rpy="0.0 0.0 3.1416" />
     </joint>
     <!-- Describe the location of the palm -->

Commit message: Millrace furtniture distances upgrade

File: urdf/ur5e_robot.urdf.xacro (robot description, xacro)
@@ -29,5 +29,5 @@
     <parent link="world" />
     <child link="small_table" />
-    <origin xyz="-0.23 -1.335 0" rpy="0 0 1.5708" />
+    <origin xyz="-0.28 -1.31 0" rpy="0 0 1.5708" />
         <!-- x_offset = 1.715 - 1.845 = -.23  distances from next wall -->
         <!-- y_offset = -1.335 -->

Commit message: f

File: urdf/ur5e_robot.urdf.xacro (robot description, xacro)
@@ -29,7 +29,11 @@
     <parent link="world" />
     <child link="small_table" />
-    <origin xyz="-0.28 -1.31 0" rpy="0 0 1.5708" />
+    <origin xyz="-0.11 -1.16 +0.24" rpy="0 0 1.5708" />
         <!-- x_offset = 1.715 - 1.845 = -.23  distances from next wall -->
         <!-- y_offset = -1.335 -->
+        <!-- Media Fellowship setup -->
+        <!-- xyz="-0.11 -1.16 +0.24" rpy="0 0 1.5708"-->
+        <!-- Fenced area setup -->
+        <!-- xyz="-0.28 -1.31 0" rpy="0 0 1.5708"-->
     </joint>
     <!-- Describe the interface between the world and the Apple Proxy -->
@@ -37,5 +41,9 @@
     <parent link = "big_table" /> -->
     <child link = "apple_proxy" /> -->
-    <origin xyz = "0.09 0.81 0.975" rpy="1.5708 0 -1.5708" />
+    <origin xyz = "0.09 0.75 0.975" rpy="1.5708 0 -1.5708" />
+        <!-- Media Fellowship setup -->
+        <!-- xyz="+0.09 +0.75 0.975" rpy="1.5708 0 -1.5708"-->
+        <!-- Fenced area setup -->
+        <!-- xyz="+0.09 +0.81 0.975" rpy="1.5708 0 -1.5708"-->
     </joint>
     <!-- Describe the interface between the world and the robot" -->

Commit message: Media Fellowship scene update

File: urdf/ur5e_robot.urdf.xacro (robot description, xacro)
@@ -29,9 +29,9 @@
     <parent link="world" />
     <child link="small_table" />
-    <origin xyz="-0.11 -1.16 +0.24" rpy="0 0 1.5708" />
+    <origin xyz="-0.11 -1.41 +0.24" rpy="0 0 1.5708" />
         <!-- x_offset = 1.715 - 1.845 = -.23  distances from next wall -->
         <!-- y_offset = -1.335 -->
         <!-- Media Fellowship setup -->
-        <!-- xyz="-0.11 -1.16 +0.24" rpy="0 0 1.5708"-->
+        <!-- xyz="-0.11 -1.41 +0.24" rpy="0 0 1.5708"-->
         <!-- Fenced area setup -->
         <!-- xyz="-0.28 -1.31 0" rpy="0 0 1.5708"-->

Commit message: Updated urdf.xacro with the scene at Millrace - Fenced Area

File: urdf/ur5e_robot.urdf.xacro (robot description, xacro)
@@ -29,11 +29,11 @@
     <parent link="world" />
     <child link="small_table" />
-    <origin xyz="-0.11 -1.41 +0.24" rpy="0 0 1.5708" />
-        <!-- x_offset = 1.715 - 1.845 = -.23  distances from next wall -->
-        <!-- y_offset = -1.335 -->
+    <origin xyz="-0.29 -1.31 +0.24" rpy="0 0 1.5708" />
+        <!-- x_offset = 1.56 - 1.85 = -.29  distances from next wall -->
+        <!-- y_offset = -1.31 -->
         <!-- Media Fellowship setup -->
         <!-- xyz="-0.11 -1.41 +0.24" rpy="0 0 1.5708"-->
         <!-- Fenced area setup -->
-        <!-- xyz="-0.28 -1.31 0" rpy="0 0 1.5708"-->
+        <!-- xyz="-0.29 -1.31 0" rpy="0 0 1.5708"-->
     </joint>
     <!-- Describe the interface between the world and the Apple Proxy -->
@@ -41,9 +41,9 @@
     <parent link = "big_table" /> -->
     <child link = "apple_proxy" /> -->
-    <origin xyz = "0.4572 0.75 0.975" rpy="1.5708 0 -1.5708" />
+    <origin xyz = "0.4572 0.91 0.975" rpy="1.5708 0 -1.5708" />
         <!-- Media Fellowship setup -->
         <!-- xyz="+0.4572 +0.75 0.975" rpy="1.5708 0 -1.5708"-->
         <!-- Fenced area setup -->
-        <!-- xyz="+0.09 +0.81 0.975" rpy="1.5708 0 -1.5708"-->
+        <!-- xyz="+0.4572 +0.91 0.975" rpy="1.5708 0 -1.5708"-->
     </joint>
     <!-- Describe the interface between the world and the robot" -->
