Commit message: Updated scene_B with the new mesh files

File: urdf/scene_B.xacro (robot description, xacro)
@@ -40,5 +40,5 @@
         <origin xyz="0 0 0" rpy="0 0 0"/>
         <geometry>
-          <mesh filename="package://apple_proxy/meshes/furniture/collision/UR5_simpleProxy.STL" scale="0.001 0.001 0.001"/>
+          <mesh filename="package://apple_proxy/meshes/apple_proxy/visual/apple_proxy_visual.STL" scale="0.001 0.001 0.001"/>
         </geometry>
         <material name="Green">
@@ -49,5 +49,5 @@
         <origin xyz="0 0 0" rpy="0 0 0"/>
         <geometry>
-          <mesh filename="package://apple_proxy/meshes/furniture/collision/UR5_simpleProxy.STL" scale="0.001 0.001 0.001"/>
+          <mesh filename="package://apple_proxy/meshes/apple_proxy/collision/apple_proxy_collision.STL" scale="0.001 0.001 0.001"/>
         </geometry>
       </collision>

Commit message: Update for the Media Fellowship Scene

File: urdf/scene_B.xacro (robot description, xacro)
@@ -38,5 +38,5 @@
     <link name="apple_proxy">
       <visual>
-        <origin xyz="0 0 0" rpy="0 0 0"/>
+        <origin xyz="-0.11498 0.7701 0" rpy="0 0 -1.5708"/>
         <geometry>
           <mesh filename="package://apple_proxy/meshes/apple_proxy/visual/apple_proxy_visual.STL" scale="0.001 0.001 0.001"/>

File: urdf/ur5e_robot.urdf.xacro (robot description, xacro)
@@ -41,7 +41,7 @@
     <parent link = "big_table" /> -->
     <child link = "apple_proxy" /> -->
-    <origin xyz = "0.09 0.75 0.975" rpy="1.5708 0 -1.5708" />
+    <origin xyz = "0.4572 0.75 0.975" rpy="1.5708 0 -1.5708" />
         <!-- Media Fellowship setup -->
-        <!-- xyz="+0.09 +0.75 0.975" rpy="1.5708 0 -1.5708"-->
+        <!-- xyz="+0.4572 +0.75 0.975" rpy="1.5708 0 -1.5708"-->
         <!-- Fenced area setup -->
         <!-- xyz="+0.09 +0.81 0.975" rpy="1.5708 0 -1.5708"-->

Commit message: Added joe's ur5 table mesh

File: urdf/scene_B.xacro (robot description, xacro)
@@ -33,4 +33,21 @@
         <geometry>
           <mesh filename="package://apple_proxy/meshes/furniture/collision/UR5_small_table.STL" scale="0.001 0.001 0.001"/>
+        </geometry>
+      </collision>
+    </link>
+    <link name="joes_ur5_table" >
+      <visual>
+        <origin xyz="0 0 0" rpy="0 0 0"/>
+        <geometry>
+          <mesh filename="package://apple_proxy/meshes/furniture/collision/joes_ur5_table.STL" scale="0.001 0.001 0.001"/>
+        </geometry>
+        <material name="Grey">
+          <color rgba="0.5 0.5 0.5 1.0"/>
+        </material>
+      </visual>
+      <collision>
+        <origin xyz="0 0 0" rpy="0 0 0"/>
+        <geometry>
+          <mesh filename="package://apple_proxy/meshes/furniture/collision/joes_ur5_table.STL" scale="0.001 0.001 0.001"/>
         </geometry>
       </collision>

Commit message: Created scene_c.xacro with joe's ur5 table mesh

File: urdf/scene_B.xacro (robot description, xacro)
@@ -33,21 +33,4 @@
         <geometry>
           <mesh filename="package://apple_proxy/meshes/furniture/collision/UR5_small_table.STL" scale="0.001 0.001 0.001"/>
-        </geometry>
-      </collision>
-    </link>
-    <link name="joes_ur5_table" >
-      <visual>
-        <origin xyz="0 0 0" rpy="0 0 0"/>
-        <geometry>
-          <mesh filename="package://apple_proxy/meshes/furniture/collision/joes_ur5_table.STL" scale="0.001 0.001 0.001"/>
-        </geometry>
-        <material name="Grey">
-          <color rgba="0.5 0.5 0.5 1.0"/>
-        </material>
-      </visual>
-      <collision>
-        <origin xyz="0 0 0" rpy="0 0 0"/>
-        <geometry>
-          <mesh filename="package://apple_proxy/meshes/furniture/collision/joes_ur5_table.STL" scale="0.001 0.001 0.001"/>
         </geometry>
       </collision>
