Commit message: Suction_Experiment meshes

File: urdf/scene_C.xacro (robot description, xacro)
@@ -19,21 +19,4 @@
       </collision>
     </link>
-    <link name="small_table" >
-      <visual>
-        <origin xyz="0 0 0" rpy="0 0 0"/>
-        <geometry>
-          <mesh filename="package://apple_proxy/meshes/furniture/collision/UR5_small_table.STL" scale="0.001 0.001 0.001"/>
-        </geometry>
-        <material name="Grey">
-          <color rgba="0.5 0.5 0.5 1.0"/>
-        </material>
-      </visual>
-      <collision>
-        <origin xyz="0 0 0" rpy="0 0 0"/>
-        <geometry>
-          <mesh filename="package://apple_proxy/meshes/furniture/collision/UR5_small_table.STL" scale="0.001 0.001 0.001"/>
-        </geometry>
-      </collision>
-    </link>
     <link name="joes_ur5_table" >
       <visual>
@@ -53,36 +36,35 @@
       </collision>
     </link>
-    <link name="apple_proxy">
+    <link name="sphere" >
       <visual>
-        <origin xyz="-0.11498 0.7701 0" rpy="0 0 -1.5708"/>
+        <origin xyz="0 0 0" rpy="0 0 0"/>
         <geometry>
-          <mesh filename="package://apple_proxy/meshes/apple_proxy/visual/apple_proxy_visual.STL" scale="0.001 0.001 0.001"/>
+          <mesh filename="package://apple_proxy/meshes/suction_experiment/sphere_base_75mm.STL" scale="0.001 0.001 0.001"/>
         </geometry>
-        <material name="Green">
-          <color rgba="0 1 0 0.7"/>
-        </material>
+        <material name="Grey">
+          <color rgba="0.5 0.5 0.5 1.0"/>
+        </material?
       </visual>
       <collision>
         <origin xyz="0 0 0" rpy="0 0 0"/>
         <geometry>
-          <mesh filename="package://apple_proxy/meshes/apple_proxy/collision/apple_proxy_collision.STL" scale="0.001 0.001 0.001"/>
+          <mesh filename="package://apple_proxy/meshes/suction_experiment/sphere_base_75mm.STL" scale="0.001 0.001 0.001"/>
         </geometry>
       </collision>
     </link>
-    <!-- Simplified Version of Lisa's hand -->
-    <link name="lisas_hand">
+    <link name="test_rig" >
       <visual>
         <origin xyz="0 0 0" rpy="0 0 0"/>
         <geometry>
-          <mesh filename="package://apple_proxy/meshes/hand/hand_cylinder.STL" scale="0.001 0.001 0.001"/>
+          <mesh filename="package://apple_proxy/meshes/suction_experiment/experiment_1_1cup_body.STL" scale="0.001 0.001 0.001"/>
         </geometry>
-        <material name="Black">
-          <color rgba="0 0 0 0.5"/>
-        </material>
+        <material name="Grey">
+          <color rgba="0.5 0.5 0.5 1.0"/>
+        </material?
       </visual>
       <collision>
         <origin xyz="0 0 0" rpy="0 0 0"/>
         <geometry>
-          <mesh filename="package://apple_proxy/meshes/hand/hand_cylinder.STL" scale="0.001 0.001 0.001"/>
+          <mesh filename="package://apple_proxy/meshes/suction_experiment/experiment_1_1cup_body.STL" scale="0.001 0.001 0.001"/>
         </geometry>
       </collision>

Commit message: scene setup

File: urdf/scene_C.xacro (robot description, xacro)
@@ -44,5 +44,5 @@
         <material name="Grey">
           <color rgba="0.5 0.5 0.5 1.0"/>
-        </material?
+        </material>
       </visual>
       <collision>
@@ -61,5 +61,5 @@
         <material name="Grey">
           <color rgba="0.5 0.5 0.5 1.0"/>
-        </material?
+        </material>
       </visual>
       <collision>

Commit message: Adjusted collision model for suction rig

File: urdf/scene_C.xacro (robot description, xacro)
@@ -40,5 +40,5 @@
         <origin xyz="0 0 0" rpy="0 0 0"/>
         <geometry>
-          <mesh filename="package://apple_proxy/meshes/suction_experiment/sphere_base_75mm.STL" scale="0.001 0.001 0.001"/>
+          <mesh filename="package://apple_proxy/meshes/suction_experiment/visual/sphere_base_75mm.STL" scale="0.001 0.001 0.001"/>
         </geometry>
         <material name="Grey">
@@ -49,5 +49,5 @@
         <origin xyz="0 0 0" rpy="0 0 0"/>
         <geometry>
-          <mesh filename="package://apple_proxy/meshes/suction_experiment/sphere_base_75mm.STL" scale="0.001 0.001 0.001"/>
+          <mesh filename="package://apple_proxy/meshes/suction_experiment/visual/sphere_base_75mm.STL" scale="0.001 0.001 0.001"/>
         </geometry>
       </collision>
@@ -57,5 +57,5 @@
         <origin xyz="0 0 0" rpy="0 0 0"/>
         <geometry>
-          <mesh filename="package://apple_proxy/meshes/suction_experiment/experiment_1_1cup_body.STL" scale="0.001 0.001 0.001"/>
+          <mesh filename="package://apple_proxy/meshes/suction_experiment/visual/experiment_1_1cup_body.STL" scale="0.001 0.001 0.001"/>
         </geometry>
         <material name="Grey">
@@ -64,7 +64,7 @@
       </visual>
       <collision>
-        <origin xyz="0 0 0" rpy="0 0 0"/>
+        <origin xyz="-0.025 0 0.085" rpy="-1.5708 0 0"/>
         <geometry>
-          <mesh filename="package://apple_proxy/meshes/suction_experiment/experiment_1_1cup_body.STL" scale="0.001 0.001 0.001"/>
+          <mesh filename="package://apple_proxy/meshes/suction_experiment/collision/suction_rig_collision_model.STL" scale="0.001 0.001 0.001"/>
         </geometry>
       </collision>

Commit message: Added suction cup in the scene for visualization

File: urdf/scene_C.xacro (robot description, xacro)
@@ -70,4 +70,21 @@
       </collision>
     </link>
+    <link name="suction_cup_model" >
+      <visual>
+        <origin xyz="0 0 0" rpy="0 0 0"/>
+        <geometry>
+          <mesh filename="package://apple_proxy/meshes/suction_experiment/visual/suction_cup_fbx20_visual.STL" scale="0.001 0.001 0.001"/>
+        </geometry>
+        <material name="Blue">
+          <color rgba="0 0 1.0 1.0"/>
+        </material>
+      </visual>
+      <collision>
+        <origin xyz="0.004 0.029 0" rpy="1.5708 0 0"/>
+        <geometry>
+          <mesh filename="package://apple_proxy/meshes/suction_experiment/collision/suction_cup_fbx20_collision.STL" scale="0.001 0.001 0.001"/>
+        </geometry>
+      </collision>
+    </link>
   </xacro:macro>
 </robot>

File: urdf/ur5e_robot_suction.urdf.xacro (robot description, xacro)
@@ -17,5 +17,5 @@
     <parent link="tool0" />
     <child link="test_rig" />
-    <origin xyz="-0.025 0.04 0" rpy="1.5708 0 0" />
+    <origin xyz="-0.026 -0.039 0.175" rpy="-1.5708 0 0" />
         <!-- Note: x and y offset is because the cframe of the 3d model is not located in the center -->
     </joint>
@@ -49,3 +49,9 @@
     <origin xyz="0 0 0.203" rpy="0 0 0" />
     </joint>
+    <!-- Describe the location of the tip of the suction cup -->
+    <joint name="suction_cup_model" type="fixed">
+    <parent link="tool0" />
+    <child link="suction_cup_model" />
+    <origin xyz="-0.0165 0.0165 0.203" rpy="3.1416 0 0" />
+    </joint>
 </robot>

Commit message: red sphere

File: urdf/scene_C.xacro (robot description, xacro)
@@ -42,6 +42,6 @@
           <mesh filename="package://apple_proxy/meshes/suction_experiment/visual/sphere_base_75mm.STL" scale="0.001 0.001 0.001"/>
         </geometry>
-        <material name="Grey">
-          <color rgba="0.5 0.5 0.5 1.0"/>
+        <material name="Red">
+          <color rgba="1 0 0 1"/>
         </material>
       </visual>

Commit message: added virtual walls to avoid werid waypoints

File: urdf/scene_C.xacro (robot description, xacro)
@@ -87,4 +87,21 @@
       </collision>
     </link>
+    <link name="virtual_walls" >
+      <visual>
+        <origin xyz="0 0 0" rpy="0 0 0"/>
+        <geometry>
+          <mesh filename="package://apple_proxy/meshes/suction_experiment/collision/imaginary_walls.STL" scale="0.001 0.001 0.001"/>
+        </geometry>
+        <material name="Blue">
+          <color rgba="0 0 1.0 0.1"/>
+        </material>
+      </visual>
+      <collision>
+        <origin xyz="0 0 0" rpy="0 0 0"/>
+        <geometry>
+          <mesh filename="package://apple_proxy/meshes/suction_experiment/collision/imaginary_walls.STL" scale="0.001 0.001 0.001"/>
+        </geometry>
+      </collision>
+    </link>
   </xacro:macro>
 </robot>

File: urdf/ur5e_robot_suction.urdf.xacro (robot description, xacro)
@@ -55,3 +55,9 @@
     <origin xyz="-0.0165 0.0165 0.203" rpy="3.1416 0 0" />
     </joint>
+    <!-- Describe the location of virtual walls -->
+    <joint name="walls" type="fixed">
+    <parent link="joes_ur5_table" />
+    <child link="virtual_walls" />
+    <origin xyz="0.9 -0.2 -0.9" rpy="0 0 1.5708" />
+    </joint>
 </robot>

Commit message: simply set joint limits to avoid weird poses

File: urdf/scene_C.xacro (robot description, xacro)
@@ -87,21 +87,4 @@
       </collision>
     </link>
-    <link name="virtual_walls" >
-      <visual>
-        <origin xyz="0 0 0" rpy="0 0 0"/>
-        <geometry>
-          <mesh filename="package://apple_proxy/meshes/suction_experiment/collision/imaginary_walls.STL" scale="0.001 0.001 0.001"/>
-        </geometry>
-        <material name="Blue">
-          <color rgba="0 0 1.0 0.1"/>
-        </material>
-      </visual>
-      <collision>
-        <origin xyz="0 0 0" rpy="0 0 0"/>
-        <geometry>
-          <mesh filename="package://apple_proxy/meshes/suction_experiment/collision/imaginary_walls.STL" scale="0.001 0.001 0.001"/>
-        </geometry>
-      </collision>
-    </link>
   </xacro:macro>
 </robot>

File: urdf/ur5e_robot_suction.urdf.xacro (robot description, xacro)
@@ -55,9 +55,3 @@
     <origin xyz="-0.0165 0.0165 0.203" rpy="3.1416 0 0" />
     </joint>
-    <!-- Describe the location of virtual walls -->
-    <joint name="walls" type="fixed">
-    <parent link="joes_ur5_table" />
-    <child link="virtual_walls" />
-    <origin xyz="0.9 -0.2 -0.8" rpy="0 0 1.5708" />
-    </joint>
 </robot>
