Commit message: scene setup

File: urdf/ur5e_robot_suction.urdf.xacro (robot description, xacro)
@@ -16,5 +16,5 @@
     <joint name="robotiq_coupler_joint" type="fixed">
     <parent link="tool0" />
-    <child link="lisas_hand" />
+    <child link="test_rig" />
     <origin xyz="-0.0675 0.0675 0.004" rpy="0 0 ${-pi/2.0}" />
         <!-- Note: x and y offset is because the cframe of the 3d model is not located in the center -->
@@ -28,26 +28,16 @@
     <joint name="world_small_table" type="fixed">
     <parent link="world" />
-    <child link="small_table" />
-    <origin xyz="-0.29 -1.31 +0.24" rpy="0 0 1.5708" />
-        <!-- x_offset = 1.56 - 1.85 = -.29  distances from next wall -->
-        <!-- y_offset = -1.31 -->
-        <!-- Media Fellowship setup -->
-        <!-- xyz="-0.11 -1.41 +0.24" rpy="0 0 1.5708"-->
-        <!-- Fenced area setup -->
-        <!-- xyz="-0.29 -1.31 0" rpy="0 0 1.5708"-->
+    <child link="joes_ur5_table" />
+    <origin xyz="0 0 0" rpy="0 0 0" />
     </joint>
-    <!-- Describe the interface between the world and the Apple Proxy -->
+    <!-- Describe the interface between the world and the Semi sphere -->
     <joint name = "bigTable_simpleProxy" type="fixed"> -->
     <parent link = "big_table" /> -->
-    <child link = "apple_proxy" /> -->
-    <origin xyz = "0.4572 0.91 0.975" rpy="1.5708 0 -1.5708" />
-        <!-- Media Fellowship setup -->
-        <!-- xyz="+0.4572 +0.75 0.975" rpy="1.5708 0 -1.5708"-->
-        <!-- Fenced area setup -->
-        <!-- xyz="+0.4572 +0.91 0.975" rpy="1.5708 0 -1.5708"-->
+    <child link = "sphere" /> -->
+    <origin xyz = "0 0 0" rpy="0 0 0" />
     </joint>
     <!-- Describe the interface between the world and the robot" -->
     <joint name="world_joint" type="fixed">
-    <parent link="small_table" />
+    <parent link="joes_ur5_table" />
     <child link = "base_link" />
     <origin xyz="0.358 0.357 0.858" rpy="0.0 0.0 3.1416" />

Commit message: scene setup

File: urdf/ur5e_robot_suction.urdf.xacro (robot description, xacro)
@@ -7,5 +7,5 @@
     <xacro:include filename="$(find ur_description)/urdf/ur5e.xacro" />
     <!--  Tables and Walls -->
-    <xacro:include filename="$(find apple_proxy)/urdf/scene_B.xacro" />
+    <xacro:include filename="$(find apple_proxy)/urdf/scene_C.xacro" />
     <xacro:tables />
     <!-- STEP 2: DEFINE THE INTERFACES AMONG ALL THE LINKS FROM -->
@@ -17,5 +17,5 @@
     <parent link="tool0" />
     <child link="test_rig" />
-    <origin xyz="-0.0675 0.0675 0.004" rpy="0 0 ${-pi/2.0}" />
+    <origin xyz="-0.025 0.04 0" rpy="1.5708 0 0" />
         <!-- Note: x and y offset is because the cframe of the 3d model is not located in the center -->
     </joint>
@@ -29,5 +29,5 @@
     <parent link="world" />
     <child link="joes_ur5_table" />
-    <origin xyz="0 0 0" rpy="0 0 0" />
+    <origin xyz="1.03 0 0.76" rpy="-3.1416 0 3.1416" />
     </joint>
     <!-- Describe the interface between the world and the Semi sphere -->
@@ -35,5 +35,5 @@
     <parent link = "big_table" /> -->
     <child link = "sphere" /> -->
-    <origin xyz = "0 0 0" rpy="0 0 0" />
+    <origin xyz = "0.115 0 1.0325" rpy="0 3.1416 0" />
     </joint>
     <!-- Describe the interface between the world and the robot" -->
@@ -41,5 +41,5 @@
     <parent link="joes_ur5_table" />
     <child link = "base_link" />
-    <origin xyz="0.358 0.357 0.858" rpy="0.0 0.0 3.1416" />
+    <origin xyz="0.71 0.25 0" rpy="3.1416 0.0 -0.7854" />
     </joint>
     <!-- Describe the location of the palm -->

Commit message: scene setup

File: urdf/ur5e_robot_suction.urdf.xacro (robot description, xacro)
@@ -12,5 +12,4 @@
     <!-- Here is where you define the scene and how the cframes are related -->
     <link name="world" />
-    <link name="palm" />
     <!-- Describe the interface between the robot and the gripper -->
     <joint name="robotiq_coupler_joint" type="fixed">
@@ -43,10 +42,3 @@
     <origin xyz="0.71 0.25 0" rpy="3.1416 0.0 -0.7854" />
     </joint>
-    <!-- Describe the location of the palm -->
-    <joint name="hand_palm" type="fixed">
-    <parent link="tool0" />
-    <child link="palm" />
-<!--        <origin xyz="0 0 0.13" rpy="0 0 0.2618 " />      &lt;!&ndash; Add in Z the hand's thickness (approx 13cm) &ndash;&gt;-->
-    <origin xyz="0 0 0.165" rpy="0 0 0.2618 " />      <!-- Add in Z the hand's thickness (approx 13cm) -->
-    </joint>
 </robot>

Commit message: setting up srdf and xacro for Suction

File: urdf/ur5e_robot_suction.urdf.xacro (robot description, xacro)
@@ -12,4 +12,5 @@
     <!-- Here is where you define the scene and how the cframes are related -->
     <link name="world" />
+    <link name="suction_cup" />
     <!-- Describe the interface between the robot and the gripper -->
     <joint name="robotiq_coupler_joint" type="fixed">
@@ -42,3 +43,9 @@
     <origin xyz="0.71 0.25 0" rpy="3.1416 0.0 -0.7854" />
     </joint>
+    <!-- Describe the location of the tip of the suction cup -->
+    <joint name="suction_cup" type="fixed">
+    <parent link="tool0" />
+    <child link="suction_cup" />
+    <origin xyz="0 0 0.203" rpy="0 0 0" />
+    </joint>
 </robot>

Commit message: calibration of suctino scene

File: urdf/ur5e_robot_suction.urdf.xacro (robot description, xacro)
@@ -29,5 +29,5 @@
     <parent link="world" />
     <child link="joes_ur5_table" />
-    <origin xyz="1.03 0 0.76" rpy="-3.1416 0 3.1416" />
+    <origin xyz="1.019 0.036 0.762" rpy="-3.1416 0 3.1416" />
     </joint>
     <!-- Describe the interface between the world and the Semi sphere -->

Commit message: calibrated urdf

File: urdf/ur5e_robot_suction.urdf.xacro (robot description, xacro)
@@ -29,5 +29,5 @@
     <parent link="world" />
     <child link="joes_ur5_table" />
-    <origin xyz="1.019 0.036 0.762" rpy="-3.1416 0 3.1416" />
+    <origin xyz="1.019 0.036 0.7670" rpy="-3.1416 0 3.1416" />
     </joint>
     <!-- Describe the interface between the world and the Semi sphere -->

Commit message: scen adjustsed

File: urdf/ur5e_robot_suction.urdf.xacro (robot description, xacro)
@@ -29,5 +29,5 @@
     <parent link="world" />
     <child link="joes_ur5_table" />
-    <origin xyz="1.019 0.036 0.7670" rpy="-3.1416 0 3.1416" />
+    <origin xyz="1.019 0.036 0.7660" rpy="-3.1416 0 3.1416" />
     </joint>
     <!-- Describe the interface between the world and the Semi sphere -->

Commit message: virtual walls

File: urdf/ur5e_robot_suction.urdf.xacro (robot description, xacro)
@@ -59,5 +59,5 @@
     <parent link="joes_ur5_table" />
     <child link="virtual_walls" />
-    <origin xyz="0.9 -0.2 -0.9" rpy="0 0 1.5708" />
+    <origin xyz="0.9 -0.2 -0.8" rpy="0 0 1.5708" />
     </joint>
 </robot>

Commit message: fixed topic to the new package

File: urdf/ur5e_robot_suction.urdf.xacro (robot description, xacro)
@@ -29,5 +29,5 @@
     <parent link="world" />
     <child link="joes_ur5_table" />
-    <origin xyz="1.019 0.036 0.7660" rpy="-3.1416 0 3.1416" />
+    <origin xyz="0.915 0.097 0.7660" rpy="-3.1416 0 3.1416" />
     </joint>
     <!-- Describe the interface between the world and the Semi sphere -->
